File: avrnote-uno.kicad_pcb (KiCad board)
At the start: 2 copper layers, 68.6 x 53.3 mm, 46 parts, among them J1 VCCSEL, J2 DC, J3 USB_C_Recept_USB2.0, J4 Power, J5 Digital/PWM, J6 Analog, J7 Digital/PWM, U1 AZ1117CH2-3.3, U2 NJM7805SDL1, U3 CH340E, U4 74AHC1G125, U5 ATmega328P-P, Y1 16MHz

Commit message: minorfix
Parts:
- Y1: footprint Crystal:Crystal_HC18-U_Vertical -> ATS08A-E:XTAL_HC49P488W43L1085T450H368
- moved Y1 2.45 mm to (141.7, 68.9)
- renumbered L to D2, ICSP to ICSP1, Reset to SW1
Routing:
- net /Vin: track 63.5 -> 65.8 mm
- net +5V: track 182.1 -> 184.0 mm
- net +3V3: track 49.5 -> 51.1 mm
- net Net-(D1-A): track 9.94 -> 10.7 mm
