File: avrnote-uno.kicad_pcb (KiCad board)
At the start: 2 copper layers, 68.6 x 53.3 mm, 46 parts, among them J1 VCCSEL, J2 DC, J3 USB_C_Recept_USB2.0, J4 Power, J5 Digital/PWM, J6 Analog, J7 Digital/PWM, SW1 SW_Reset, U1 AZ1117CH2-3.3, U2 NJM7805SDL1, U3 CH340E, U4 74AHC1G125, U5 ATmega328P-P, Y1 16MHz

Commit message: fix: az1117ch2-3.3v -> az1117ch-3.3v
Parts:
- U1: value AZ1117CH2-3.3 -> AZ1117CH-3.3TRG1; footprint Package_TO_SOT_SMD:SOT-223-3_TabPin2 -> AZ1117CH-3.3TRG1:VREG_AZ1117CH-3.3TRG1
- moved U1 4.10 mm to (105.6, 74.6)
- moved C2 3.85 mm to (117.3, 71.6)
- moved F1 2.67 mm to (115.5, 75.4)
- moved R1 2.65 mm to (106.1, 61.4), turned to 0 degrees
- moved C6 1.44 mm to (116.8, 81.2)
- moved U2 1.11 mm to (105.8, 82.5)
Connections:
- U1 pad 1: +5V -> GND
- U1 pad 2: GND -> +3V3
- U1 pad 3: +3V3 -> +5V
Routing:
- net +3V3: track 51.1 -> 54.6 mm
- net /UVCC: track 10.9 -> 8.02 mm
- net Net-(F1-Pad1): track 33.5 -> 36.3 mm
- net /Vin: track 65.8 -> 63.7 mm
- net +5V: track 184.0 -> 185.9 mm
- net Net-(J3-CC2): track 8.14 -> 8.71 mm
- net GND: vias 32 -> 31

Commit message: refactor
Parts:
- F1: footprint Inductor_SMD:L_TechFuse_SL0420 -> Fuse:Fuse_1206_3216Metric
- R10: footprint Resistor_THT:R_Axial_DIN0204_L3.6mm_D1.6mm_P5.08mm_Horizontal -> Resistor_SMD:R_0603_1608Metric
- moved R4 51.0 mm to (112.7, 53.8), turned to 90 degrees
- moved R5 47.1 mm to (114.7, 53.8), turned to 90 degrees
- moved SW1 46.0 mm to (109.3, 54.5)
- moved D3 44.2 mm to (115.5, 56.6), turned to 180 degrees
- moved C9 17.5 mm to (106.9, 70.0), turned to 180 degrees
- moved C5 9.17 mm to (116.0, 62.7), turned to 180 degrees
- moved R1 9.10 mm to (103.2, 70.0), turned to 180 degrees
- moved R2 8.37 mm to (110.4, 58.8)
- moved U3 8.19 mm to (114.7, 65.5)
- moved J3 8.04 mm to (103.5, 63.1)
- moved D2 7.15 mm to (113.9, 68.8)
- moved R3 7.03 mm to (117.2, 68.8)
- moved C10 3.82 mm to (119.0, 57.8), turned to 0 degrees
- moved R10 2.62 mm to (141.7, 74.1)
- moved C11 2.50 mm to (144.4, 66.2)
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- renumbered ICSP1 to ICSP
Routing:
- net /~{RESET}: track 80.1 -> 146.2 mm, vias 0 -> 6
- net Net-(F1-Pad1): track 36.3 -> 20.5 mm
- net +5V: track 185.9 -> 194.5 mm, vias 0 -> 2
- net Net-(U3-TXD): track 46.7 -> 52.3 mm
- net Net-(J3-CC2): track 8.71 -> 10.9 mm
- net GND: track 5.95 -> 8.11 mm, vias 31 -> 40
- net /13: track 94.5 -> 96.4 mm
- net Net-(U3-RXD): track 48.0 -> 46.3 mm
- net Net-(U3-TNOW): track 3.86 -> 2.80 mm
- net Net-(U3-UD-): track 11.7 -> 12.7 mm, vias 2 -> 0
- net Net-(J3-CC1): track 4.00 -> 4.71 mm
- net Net-(U3-V3): track 2.34 -> 2.93 mm
- net /XTAL2: track 13.5 -> 12.9 mm, vias 0 -> 1
- net Net-(D2-A): track 2.16 -> 1.65 mm
- net /XTAL1: track 14.6 -> 14.1 mm, vias 0 -> 1
Other:
- board text added: "L"
- board text added: "Reset"
